Commit message: Simplified launch files and models

File: thymio_driver/models/base.urdf.xacro (robot description, xacro)
@@ -1,21 +1,21 @@
 <?xml version="1.0"?>
-<robot name="myfirst">
+<robot xmlns:xacro="http://ros.org/wiki/xacro">
+<xacro:macro name="thymio">
   <link name="base_link">
     <visual>
       <geometry>
 	<mesh filename="package://thymio_driver/models/meshes/thymio.dae"/>
-        <!--><cylinder length="0.1" radius="0.2"/><-->
       </geometry>
     </visual>
   </link>
- <link name="proximity_center_link"/>
- <link name="proximity_center_left_link"/>
- <link name="proximity_center_right_link"/>
- <link name="proximity_left_link"/>
- <link name="proximity_right_link"/>
- <link name="proximity_rear_left_link"/>
- <link name="proximity_rear_right_link"/>
- <link name="ground_left_link"/>
- <link name="ground_right_link"/>
+  <link name="proximity_center_link"/>
+  <link name="proximity_center_left_link"/>
+  <link name="proximity_center_right_link"/>
+  <link name="proximity_left_link"/>
+  <link name="proximity_right_link"/>
+  <link name="proximity_rear_left_link"/>
+  <link name="proximity_rear_right_link"/>
+  <link name="ground_left_link"/>
+  <link name="ground_right_link"/>
   <joint name="proximity_center_joint" type="fixed">
     <origin xyz="0.08 0 0.034" rpy="0 0 0"/>
@@ -63,3 +63,4 @@
     <child link="ground_left_link"/>
   </joint>
+</xacro:macro>
 </robot>
